Commit message: Adjust model puma to real

File: puma_simulation/puma_model/urdf/puma_model.urdf (robot description, URDF)
Before this commit: robot puma_model, 8 links, 7 joints
Links:
- added link gps_link, mass 0.1; collision mesh filename=package://puma_model/meshes/gps_link.STL; visual mesh filename=package://puma_model/meshes/gps_link.STL
- added link imu1_link, mass 0.1; collision mesh filename=package://puma_model/meshes/imu1_link.STL; visual mesh filename=package://puma_model/meshes/imu1_link.STL
- added link imu2_link, mass 0.1; collision mesh filename=package://puma_model/meshes/imu2_link.STL; visual mesh filename=package://puma_model/meshes/imu2_link.STL
- link base_link: mass 137.364583550566 -> 154.38
- link dir_left_link: mass 0.45023 -> 0.214607285846125
- link dir_right_link: mass 0.45023 -> 0.21461
- link wheel_left_back_link: mass 39.8759403950152 -> 42.8421975932662
- link wheel_left_front_link: mass 32.018 -> 33.8332405777372
- link wheel_right_back_link: mass 39.8759403950152 -> 42.8421975932662
- link wheel_right_front_link: mass 32.018 -> 33.833
Joints:
- added joint gps_joint: type fixed, parent base_link, child gps_link, origin xyz=0.27173 0 0.76 rpy=0 0 0, axis 0 0 0
- added joint imu1_link: type fixed, parent base_link, child imu1_link, origin xyz=-0.74327 0 0.57 rpy=0 0 0, axis 0 0 0
- added joint imu2_joint: type fixed, parent base_link, child imu2_link, origin xyz=0.646729916214884 0 0.37 rpy=0 0 0, axis 0 0 0
- joint base_component_joint: origin xyz=0.0767267348036579 0 0.63 rpy=0 0 0 -> xyz=0.12673 0 0.63 rpy=0 0 0
- joint dir_left_joint: limit (none) -> lower=0 upper=0 effort=0 velocity=0; origin xyz=0.526726734803658 0.353 0.265 rpy=0 0 0 -> xyz=0.576729916214884 0.337 0.265 rpy=0 0 0
- joint dir_right_joint: limit (none) -> lower=0 upper=0 effort=0 velocity=0; origin xyz=0.526726734803658 -0.353 0.265 rpy=0 0 0 -> xyz=0.57673 -0.337 0.265 rpy=0 0 0
- joint wheel_left_back_joint: limit (none) -> lower=0 upper=0 effort=0 velocity=0; origin xyz=-0.523273265196342 0.275 0.249999999999999 rpy=-1.5707963267949 0 0 -> xyz=-0.57327 0.275 0.25 rpy=-1.5708 0 0
- joint wheel_left_front_joint: limit (none) -> lower=0 upper=0 effort=0 velocity=0; origin xyz=0 0.078 0 rpy=1.5707963267949 0 -3.14159265358979 -> xyz=0 0.048 0 rpy=1.5708 0 -3.1416
- joint wheel_right_back_joint: limit (none) -> lower=0 upper=0 effort=0 velocity=0; origin xyz=-0.523273265196343 -0.275 0.250000000000001 rpy=1.5707963267949 0 0 -> xyz=-0.57327 -0.275 0.25 rpy=1.5708 0 0
- joint wheel_right_front_joint: limit (none) -> lower=0 upper=0 effort=0 velocity=0; origin xyz=0 -0.0779999999999998 0 rpy=1.5707963267949 0 0 -> xyz=0 -0.048 0 rpy=1.5708 0 0

File: puma_simulation/puma_model/urdf/puma_model.urdf.xacro (robot description, xacro)
@@ -9,15 +9,15 @@
     <inertial>
       <origin
-        xyz="0.016651799447873 2.50054494388419E-07 0.3700954993344"
-        rpy="0 0 0" />
-      <mass
-        value="141.871222119219" />
-      <inertia
-        ixx="3.58592238244372"
-        ixy="-7.70630741878065E-07"
-        ixz="1.05770487262547"
-        iyy="17.6914485683265"
-        iyz="8.25132789133817E-06"
-        izz="18.0504461411871" />
+        xyz="0.016828 2.5244E-07 0.36947"
+        rpy="0 0 0" />
+      <mass
+        value="154.38" />
+      <inertia
+        ixx="3.8644"
+        ixy="-9.5023E-07"
+        ixz="1.1536"
+        iyy="22.232"
+        iyz="9.0131E-06"
+        izz="22.651" />
     </inertial>
     <visual>
@@ -32,5 +32,5 @@
         name="">
         <color
-          rgba="0.988235294117647 0.737254901960784 0.517647058823529 1" />
+          rgba="0.98824 0.73725 0.51765 1" />
       </material>
     </visual>
@@ -49,15 +49,15 @@
     <inertial>
       <origin
-        xyz="3.33066907387547E-16 -0.047021105109952 0"
-        rpy="0 0 0" />
-      <mass
-        value="0.450226734865359" />
-      <inertia
-        ixx="0.000452930170196998"
-        ixy="-2.08351206347224E-20"
-        ixz="-1.93425232022472E-21"
-        iyy="0.000507367249025541"
-        iyz="3.95205740912683E-20"
-        izz="0.000460794419124139" />
+        xyz="-2.2204E-16 -0.029478 0"
+        rpy="0 0 0" />
+      <mass
+        value="0.21461" />
+      <inertia
+        ixx="0.00016179"
+        ixy="-1.2567E-20"
+        ixz="-1.7214E-21"
+        iyy="0.00021284"
+        iyz="1.1854E-20"
+        izz="0.00016965" />
     </inertial>
     <visual>
@@ -72,5 +72,5 @@
         name="">
         <color
-          rgba="0.823529411764706 0.823529411764706 0.823529411764706 1" />
+          rgba="0.82353 0.82353 0.82353 1" />
       </material>
     </visual>
@@ -89,5 +89,5 @@
     type="continuous">
     <origin
-      xyz="0.52673 -0.353 0.265"
+      xyz="0.57673 -0.337 0.265"
       rpy="0 0 0" />
     <parent
@@ -102,15 +102,15 @@
     <inertial>
       <origin
-        xyz="0 -1.11022302462516E-16 0.0700000000000001"
-        rpy="0 0 0" />
-      <mass
-        value="33.8332405777372" />
-      <inertia
-        ixx="0.663166940004142"
-        ixy="1.74598601904134E-32"
-        ixz="4.51486827425246E-17"
-        iyy="0.663166940004142"
-        iyz="1.07735398960113E-17"
-        izz="1.19194782788173" />
+        xyz="0 1.1102E-16 0.07"
+        rpy="0 0 0" />
+      <mass
+        value="33.833" />
+      <inertia
+        ixx="0.66317"
+        ixy="1.746E-32"
+        ixz="4.5149E-17"
+        iyy="0.66317"
+        iyz="1.0774E-17"
+        izz="1.1919" />
     </inertial>
     <visual>
@@ -125,5 +125,5 @@
         name="">
         <color
-          rgba="1 0.752941176470588 0.752941176470588 1" />
+          rgba="1 0.75294 0.75294 1" />
       </material>
     </visual>
@@ -142,5 +142,5 @@
     type="continuous">
     <origin
-      xyz="0 -0.078 0"
+      xyz="0 -0.048 0"
       rpy="1.5708 0 0" />
     <parent
@@ -157,15 +157,15 @@
     <inertial>
       <origin
-        xyz="4.44089209850063E-16 0.0470211051099522 1.11022302462516E-16"
-        rpy="0 0 0" />
-      <mass
-        value="0.450226734865359" />
-      <inertia
-        ixx="0.000452930170196997"
-        ixy="-7.29252817374884E-21"
-        ixz="-1.63781186538735E-21"
-        iyy="0.00050736724902554"
-        iyz="1.60159589115665E-20"
-        izz="0.000460794419124138" />
+        xyz="0 0.0294777193153578 1.11022302462516E-16"
+        rpy="0 0 0" />
+      <mass
+        value="0.214607285846125" />
+      <inertia
+        ixx="0.000161787233745492"
+        ixy="1.7829483231954E-21"
+        ixz="-2.5363205724219E-21"
+        iyy="0.000212842937751498"
+        iyz="3.89270928347116E-20"
+        izz="0.000169651482672632" />
     </inertial>
     <visual>
@@ -197,5 +197,5 @@
     type="continuous">
     <origin
-      xyz="0.52673 0.353 0.265"
+      xyz="0.576729916214884 0.337 0.265"
       rpy="0 0 0" />
     <parent
@@ -210,5 +210,5 @@
     <inertial>
       <origin
-        xyz="0 2.22044604925031E-16 0.0700000000000002"
+        xyz="0 0 0.0699999999999999"
         rpy="0 0 0" />
       <mass
@@ -216,8 +216,8 @@
       <inertia
         ixx="0.663166940004142"
-        ixy="4.56652860083993E-32"
+        ixy="3.62902943280336E-32"
         ixz="-3.47625364951278E-17"
         iyy="0.663166940004142"
-        iyz="-9.24811874513642E-18"
+        iyz="1.01566182105979E-18"
         izz="1.19194782788173" />
     </inertial>
@@ -250,5 +250,5 @@
     type="continuous">
     <origin
-      xyz="0 0.078 0"
+      xyz="0 0.048 0"
       rpy="1.5708 0 -3.1416" />
     <parent
@@ -265,5 +265,5 @@
     <inertial>
       <origin
-        xyz="1.55431223447522E-15 -1.55431223447522E-15 0.1"
+        xyz="0 1.11022302462516E-16 0.1"
         rpy="0 0 0" />
       <mass
@@ -271,8 +271,8 @@
       <inertia
         ixx="0.843504879614984"
-        ixy="-9.59503304028305E-33"
-        ixz="6.01287397790472E-17"
+        ixy="-2.17897005442215E-32"
+        ixz="6.01287397790473E-17"
         iyy="0.843504879614984"
-        iyz="-2.42963471245841E-16"
+        iyz="-2.51058847467066E-16"
         izz="1.34196583325215" />
     </inertial>
@@ -305,5 +305,5 @@
     type="continuous">
     <origin
-      xyz="-0.52327 -0.275 0.25"
+      xyz="-0.57327 -0.275 0.25"
       rpy="1.5708 0 0" />
     <parent
@@ -320,5 +320,5 @@
     <inertial>
       <origin
-        xyz="3.33066907387547E-16 -2.22044604925031E-16 0.0999999999999999"
+        xyz="1.11022302462516E-16 1.11022302462516E-16 0.1"
         rpy="0 0 0" />
       <mass
@@ -326,8 +326,8 @@
       <inertia
         ixx="0.843504879614984"
-        ixy="-5.97993043604167E-33"
-        ixz="-3.69567293190445E-18"
+        ixy="-4.06685460585996E-33"
+        ixz="-3.69567293190446E-18"
         iyy="0.843504879614984"
-        iyz="1.50156913172873E-17"
+        iyz="1.64612942139347E-17"
         izz="1.34196583325215" />
     </inertial>
@@ -360,5 +360,5 @@
     type="continuous">
     <origin
-      xyz="-0.52327 0.275 0.25"
+      xyz="-0.57327 0.275 0.25"
       rpy="-1.5708 0 0" />
     <parent
@@ -375,5 +375,5 @@
     <inertial>
       <origin
-        xyz="0 -1.38777878078145E-17 0"
+        xyz="-1.38777878078145E-17 -1.38777878078145E-17 0"
         rpy="0 0 0" />
       <mass
@@ -381,8 +381,8 @@
       <inertia
         ixx="0.399432"
-        ixy="5.25749814054658E-17"
-        ixz="-1.90310730137829E-18"
+        ixy="1.53695574785691E-18"
+        ixz="-1.04083408558608E-17"
         iyy="0.368016"
-        iyz="5.64237288394698E-34"
+        iyz="1.04083408558608E-17"
         izz="0.5502288" />
     </inertial>
@@ -415,5 +415,5 @@
     type="fixed">
     <origin
-      xyz="0.076727 0 0.63"
+      xyz="0.12673 0 0.63"
       rpy="0 0 0" />
     <parent
@@ -428,14 +428,14 @@
     <inertial>
       <origin
-        xyz="0 0 -0.00999999999999995"
+        xyz="0 -1.38777878078145E-17 -0.01"
         rpy="0 0 0" />
       <mass
         value="0.1" />
       <inertia
-        ixx="8.66666666666667E-05"
-        ixy="1.76566841298316E-20"
-        ixz="1.00796920723262E-21"
+        ixx="8.66666666666668E-05"
+        ixy="7.16025184745641E-22"
+        ixz="-2.70628567440132E-38"
         iyy="2.41666666666667E-05"
-        iyz="-4.3548787261501E-22"
+        iyz="-4.35487872615009E-22"
         izz="0.000104166666666667" />
     </inertial>
@@ -468,5 +468,5 @@
     type="fixed">
     <origin
-      xyz="0.22173 0 0.76"
+      xyz="0.27173 0 0.76"
       rpy="0 0 0" />
     <parent
@@ -481,5 +481,5 @@
     <inertial>
       <origin
-        xyz="0.01 0 0"
+        xyz="0.01 -1.38777878078145E-17 0"
         rpy="0 0 0" />
       <mass
@@ -487,8 +487,8 @@
       <inertia
         ixx="0.000104166666666667"
-        ixy="1.57322252736699E-21"
-        ixz="2.01593841446523E-21"
+        ixy="1.2202921326777E-21"
+        ixz="7.05860789378583E-22"
         iyy="8.6666666666667E-05"
-        iyz="-1.03902708196528E-20"
+        iyz="-1.12757025938493E-20"
         izz="2.41666666666667E-05" />
     </inertial>
@@ -518,8 +518,8 @@
   </link>
   <joint
-    name="imu1_joint"
+    name="imu1_link"
     type="fixed">
     <origin
-      xyz="-0.69327 0 0.57"
+      xyz="-0.74327 0 0.57"
       rpy="0 0 0" />
     <parent
@@ -534,5 +534,5 @@
     <inertial>
       <origin
-        xyz="-0.01 0 0"
+        xyz="-0.01 0 -1.11022302462516E-16"
         rpy="0 0 0" />
       <mass
@@ -540,8 +540,8 @@
       <inertia
         ixx="0.000104166666666667"
-        ixy="-5.26402742286973E-22"
-        ixz="2.3628831096606E-21"
+        ixy="-1.73472347597681E-22"
+        ixz="1.75866627395253E-21"
         iyy="8.66666666666669E-05"
-        iyz="6.6181507612138E-22"
+        iyz="2.31296463463575E-21"
         izz="2.41666666666667E-05" />
     </inertial>
@@ -574,5 +574,5 @@
     type="fixed">
     <origin
-      xyz="0.59673 0 0.37"
+      xyz="0.646729916214884 0 0.37"
       rpy="0 0 0" />
     <parent
