Commit message: Fix default value joy and add controller puma gazebo

File: puma_simulation/puma_model/urdf/puma_model.gazebo.xacro (robot description, xacro)
@@ -6,47 +6,75 @@
     </plugin>
   </gazebo>
-   <!-- Transmisión para la rueda trasera derecha -->
-<transmission name="wheel_back_right">
-  <type>transmission_interface/SimpleTransmission</type>
-  <joint name="wheel_right_back_joint">
-    <hardwareInterface>hardware_interface/VelocityJointInterface</hardwareInterface>
-  </joint>
-  <actuator name="wheel_right_actuator">
-    <hardwareInterface>hardware_interface/VelocityJointInterface</hardwareInterface>
-    <mechanicalReduction>1</mechanicalReduction>
-  </actuator>
-</transmission>
-<!-- Transmisión para la rueda trasera izquierda -->
-<transmission name="wheel_back_left">
-  <type>transmission_interface/SimpleTransmission</type>
-  <joint name="wheel_left_back_joint">
-    <hardwareInterface>hardware_interface/VelocityJointInterface</hardwareInterface>
-  </joint>
-  <actuator name="wheel_left_actuator">
-    <hardwareInterface>hardware_interface/VelocityJointInterface</hardwareInterface>
-    <mechanicalReduction>1</mechanicalReduction>
-  </actuator>
-</transmission>
-<!-- Transmisión para la dirección izquierda -->
-<transmission name="direction_left">
-  <type>transmission_interface/SimpleTransmission</type>
-  <joint name="dir_left_joint">
+  <!-- Transmisión para la rueda trasera derecha -->
+  <transmission name="wheel_back_right">
+    <type>transmission_interface/SimpleTransmission</type>
+    <joint name="wheel_right_back_joint">
+      <hardwareInterface>hardware_interface/VelocityJointInterface</hardwareInterface>
+    </joint>
+    <actuator name="wheel_right_actuator">
+      <hardwareInterface>hardware_interface/VelocityJointInterface</hardwareInterface>
+      <mechanicalReduction>1</mechanicalReduction>
+    </actuator>
+  </transmission>
+  <!-- Transmisión para la rueda trasera izquierda -->
+  <transmission name="wheel_back_left">
+    <type>transmission_interface/SimpleTransmission</type>
+    <joint name="wheel_left_back_joint">
+      <hardwareInterface>hardware_interface/VelocityJointInterface</hardwareInterface>
+    </joint>
+    <actuator name="wheel_left_actuator">
+      <hardwareInterface>hardware_interface/VelocityJointInterface</hardwareInterface>
+      <mechanicalReduction>1</mechanicalReduction>
+    </actuator>
+  </transmission>
+  <!-- Transmisión para la dirección izquierda -->
+  <transmission name="direction_left">
+    <type>transmission_interface/SimpleTransmission</type>
+    <joint name="dir_left_joint">
+      <hardwareInterface>hardware_interface/PositionJointInterface</hardwareInterface>
+    </joint>
+    <actuator name="direction_motor_left">
+      <hardwareInterface>PositionJointInterface</hardwareInterface>
+      <mechanicalReduction>1</mechanicalReduction>
+    </actuator>
+  </transmission>
+  <!-- Transmisión para la dirección derecha -->
+  <transmission name="direction_right">
+    <type>transmission_interface/SimpleTransmission</type>
+    <joint name="dir_right_joint">
     <hardwareInterface>hardware_interface/PositionJointInterface</hardwareInterface>
-  </joint>
-  <actuator name="direction_motor_left">
-    <hardwareInterface>PositionJointInterface</hardwareInterface>
-    <mechanicalReduction>1</mechanicalReduction>
-  </actuator>
-</transmission>
-<!-- Transmisión para la dirección derecha -->
-<transmission name="direction_right">
-  <type>transmission_interface/SimpleTransmission</type>
-  <joint name="dir_right_joint">
-   <hardwareInterface>hardware_interface/PositionJointInterface</hardwareInterface>
-  </joint>
-  <actuator name="direction_motor_right">
-    <hardwareInterface>PositionJointInterface</hardwareInterface>
-    <mechanicalReduction>1</mechanicalReduction>
-  </actuator>
-</transmission>
+    </joint>
+    <actuator name="direction_motor_right">
+      <hardwareInterface>PositionJointInterface</hardwareInterface>
+      <mechanicalReduction>1</mechanicalReduction>
+    </actuator>
+  </transmission>
+  <!-- Configuracion de links -->
+  <gazebo reference="wheel_right_front_link">
+    <mu1>1</mu1>
+    <mu2>1</mu2>
+    <minDepth>0.003</minDepth>
+    <material> Gazebo/Grey </material>
+  </gazebo>
+  <gazebo reference="wheel_left_front_link">
+    <mu1>1</mu1>
+    <mu2>1</mu2>
+    <minDepth>0.003</minDepth>
+    <material> Gazebo/Grey </material>
+  </gazebo>
+  <gazebo reference="wheel_right_back_link">
+    <mu1>1</mu1>
+    <mu2>1</mu2>
+    <minDepth>0.003</minDepth>
+    <material> Gazebo/Grey </material>
+  </gazebo>
+  <gazebo reference="wheel_left_back_link">
+    <mu1>1</mu1>
+    <mu2>1</mu2>
+    <minDepth>0.003</minDepth>
+    <material>Gazebo/Grey</material>
+  </gazebo>
+  <gazebo reference="base_link">
+    <material>Gazebo/ZincYellow</material>
+  </gazebo>
 </robot>

File: puma_simulation/puma_model/urdf/puma_model.urdf.xacro (robot description, xacro)
@@ -150,4 +150,6 @@
     <axis
       xyz="0 0 -1" />
+    <dynamics
+      friction="1" />
   </joint>
   <link
@@ -256,4 +258,6 @@
     <axis
       xyz="0 0 -1" />
+    <dynamics
+      friction="1" />
   </joint>
   <link
@@ -309,4 +313,6 @@
     <axis
       xyz="0 0 -1" />
+    <dynamics
+      friction="1" />
   </joint>
   <link
@@ -362,4 +368,6 @@
     <axis
       xyz="0 0 -1" />
+    <dynamics
+      friction="1" />
   </joint>
   <link

Commit message: Regroup directory and finish puma_controller gazebo

File: puma_simulation/puma_model/urdf/puma_model.gazebo.xacro (robot description, xacro)
@@ -78,3 +78,6 @@
     <material>Gazebo/ZincYellow</material>
   </gazebo>
+  <gazebo reference="base_component_link">
+    <material>Gazebo/Turquoise  </material>
+  </gazebo>
 </robot>

Commit message: Update model & add gps, imu

File: puma_simulation/puma_model/urdf/puma_model.gazebo.xacro (robot description, xacro)
@@ -2,6 +2,39 @@
 <robot xmlns:xacro="http://www.ros.org/wiki/xacro" name="puma_model_sim">
   <gazebo>
+    <!-- Plugin ros gazebo controller -->
     <plugin name="gazebo_ros_control" filename="libgazebo_ros_control.so">
       <robotNamespace>/</robotNamespace>
+    </plugin>
+    <!-- Plugin Gps simulate (requires hector gazebo plugins) -->
+    <plugin name="gps_controller" filename="libhector_gazebo_ros_gps.so">
+      <alwayson>true</alwayson>
+      <updaterate>1.0</updaterate>
+      <bodyName>gps_link</bodyName>
+      <frameId>/world</frameId>
+      <topicName>/fix_gps</topicName>
+      <referenceLatitude>-33.42196309675523</referenceLatitude>
+      <referenceLongitude>-70.5818018059048</referenceLongitude>
+      <referenceAltitude>570</referenceAltitude>
+      <velocitytopicname>/fix_velocity</velocitytopicname>
+      <drift>5.0 5.0 5.0</drift>
+      <gaussiannoise>0.1 0.1 0.1</gaussiannoise>
+      <velocitydrift>0 0 0</velocitydrift>
+      <velocitygaussiannoise>0.1 0.1 0.1</velocitygaussiannoise>
+    </plugin>
+    <!-- Plugin IMU 1 -->
+    <plugin name="imu1_controller" filename="libhector_gazebo_ros_imu.so">
+      <updateRate>60</updateRate>
+      <bodyName>imu1_link</bodyName>
+      <topicName>/imu1</topicName>
+      <frameId>imu1_link</frameId>
+      <gaussianNoise>0.1 0.1 0.1</gaussianNoise>
+    </plugin>
+    <!-- Plugin IMU 2  -->
+    <plugin name="imu1_controller" filename="libhector_gazebo_ros_imu.so">
+      <updateRate>60</updateRate>
+      <bodyName>imu2_link</bodyName>
+      <topicName>/imu2</topicName>
+      <frameId>imu2_link</frameId>
+      <gaussianNoise>0.1 0.1 0.1</gaussianNoise>
     </plugin>
   </gazebo>

File: puma_simulation/puma_model/urdf/puma_model.urdf.xacro (robot description, xacro)
@@ -9,15 +9,15 @@
     <inertial>
       <origin
-        xyz="0.000318371260688873 2.58258248245213E-07 0.367218886964779"
-        rpy="0 0 0" />
-      <mass
-        value="137.364583550566" />
-      <inertia
-        ixx="3.48024888119141"
-        ixy="-1.35770833137747E-06"
-        ixz="1.25278348088499"
-        iyy="16.4664872890134"
-        iyz="8.1493916197498E-06"
-        izz="16.8109813346284" />
+        xyz="0.016651799447873 2.50054494388419E-07 0.3700954993344"
+        rpy="0 0 0" />
+      <mass
+        value="141.871222119219" />
+      <inertia
+        ixx="3.58592238244372"
+        ixy="-7.70630741878065E-07"
+        ixz="1.05770487262547"
+        iyy="17.6914485683265"
+        iyz="8.25132789133817E-06"
+        izz="18.0504461411871" />
     </inertial>
     <visual>
@@ -49,15 +49,15 @@
     <inertial>
       <origin
-        xyz="3.3307E-16 -0.047021 0"
-        rpy="0 0 0" />
-      <mass
-        value="0.45023" />
-      <inertia
-        ixx="0.00045293"
-        ixy="-2.0835E-20"
-        ixz="-1.9343E-21"
-        iyy="0.00050737"
-        iyz="3.9521E-20"
-        izz="0.00046079" />
+        xyz="3.33066907387547E-16 -0.047021105109952 0"
+        rpy="0 0 0" />
+      <mass
+        value="0.450226734865359" />
+      <inertia
+        ixx="0.000452930170196998"
+        ixy="-2.08351206347224E-20"
+        ixz="-1.93425232022472E-21"
+        iyy="0.000507367249025541"
+        iyz="3.95205740912683E-20"
+        izz="0.000460794419124139" />
     </inertial>
     <visual>
@@ -72,5 +72,5 @@
         name="">
         <color
-          rgba="0.82353 0.82353 0.82353 1" />
+          rgba="0.823529411764706 0.823529411764706 0.823529411764706 1" />
       </material>
     </visual>
@@ -89,5 +89,5 @@
     type="continuous">
     <origin
-      xyz="0.526726734803658 -0.353 0.265"
+      xyz="0.52673 -0.353 0.265"
       rpy="0 0 0" />
     <parent
@@ -102,15 +102,15 @@
     <inertial>
       <origin
-        xyz="0 -1.1102E-16 0.07"
-        rpy="0 0 0" />
-      <mass
-        value="32.018" />
-      <inertia
-        ixx="0.59867"
-        ixy="-3.3873E-32"
-        ixz="3.9787E-17"
-        iyy="0.59867"
-        iyz="-1.4091E-18"
-        izz="1.0783" />
+        xyz="0 -1.11022302462516E-16 0.0700000000000001"
+        rpy="0 0 0" />
+      <mass
+        value="33.8332405777372" />
+      <inertia
+        ixx="0.663166940004142"
+        ixy="1.74598601904134E-32"
+        ixz="4.51486827425246E-17"
+        iyy="0.663166940004142"
+        iyz="1.07735398960113E-17"
+        izz="1.19194782788173" />
     </inertial>
     <visual>
@@ -125,5 +125,5 @@
         name="">
         <color
-          rgba="1 0.75294 0.75294 1" />
+          rgba="1 0.752941176470588 0.752941176470588 1" />
       </material>
     </visual>
@@ -142,6 +142,6 @@
     type="continuous">
     <origin
-      xyz="0 -0.0779999999999998 0"
-      rpy="1.5707963267949 0 0" />
+      xyz="0 -0.078 0"
+      rpy="1.5708 0 0" />
     <parent
       link="dir_right_link" />
@@ -157,15 +157,15 @@
     <inertial>
       <origin
-        xyz="4.4409E-16 0.047021 1.1102E-16"
-        rpy="0 0 0" />
-      <mass
-        value="0.45023" />
-      <inertia
-        ixx="0.00045293"
-        ixy="-7.2925E-21"
-        ixz="-1.6378E-21"
-        iyy="0.00050737"
-        iyz="1.6016E-20"
-        izz="0.00046079" />
+        xyz="4.44089209850063E-16 0.0470211051099522 1.11022302462516E-16"
+        rpy="0 0 0" />
+      <mass
+        value="0.450226734865359" />
+      <inertia
+        ixx="0.000452930170196997"
+        ixy="-7.29252817374884E-21"
+        ixz="-1.63781186538735E-21"
+        iyy="0.00050736724902554"
+        iyz="1.60159589115665E-20"
+        izz="0.000460794419124138" />
     </inertial>
     <visual>
@@ -180,5 +180,5 @@
         name="">
         <color
-          rgba="0.82353 0.82353 0.82353 1" />
+          rgba="0.823529411764706 0.823529411764706 0.823529411764706 1" />
       </material>
     </visual>
@@ -197,5 +197,5 @@
     type="continuous">
     <origin
-      xyz="0.526726734803658 0.353 0.265"
+      xyz="0.52673 0.353 0.265"
       rpy="0 0 0" />
     <parent
@@ -210,15 +210,15 @@
     <inertial>
       <origin
-        xyz="0 1.1102E-16 0.07"
-        rpy="0 0 0" />
-      <mass
-        value="32.018" />
-      <inertia
-        ixx="0.59867"
-        ixy="-1.4193E-32"
-        ixz="-3.1297E-17"
-        iyy="0.59867"
-        iyz="-1.7836E-17"
-        izz="1.0783" />
+        xyz="0 2.22044604925031E-16 0.0700000000000002"
+        rpy="0 0 0" />
+      <mass
+        value="33.8332405777372" />
+      <inertia
+        ixx="0.663166940004142"
+        ixy="4.56652860083993E-32"
+        ixz="-3.47625364951278E-17"
+        iyy="0.663166940004142"
+        iyz="-9.24811874513642E-18"
+        izz="1.19194782788173" />
     </inertial>
     <visual>
@@ -233,5 +233,5 @@
         name="">
         <color
-          rgba="1 0.75294 0.75294 1" />
+          rgba="1 0.752941176470588 0.752941176470588 1" />
       </material>
     </visual>
@@ -251,5 +251,5 @@
     <origin
       xyz="0 0.078 0"
-      rpy="1.5707963267949 0 -3.14159265358979" />
+      rpy="1.5708 0 -3.1416" />
     <parent
       link="dir_left_link" />
@@ -265,15 +265,15 @@
     <inertial>
       <origin
-        xyz="1.4432899320127E-15 -1.55431223447522E-15 0.1"
-        rpy="0 0 0" />
-      <mass
-        value="39.8759403950152" />
-      <inertia
-        ixx="0.738004078739411"
-        ixy="-2.40636772622452E-32"
-        ixz="5.01473497824115E-17"
-        iyy="0.738004078739411"
-        iyz="-2.10536971222048E-16"
-        izz="1.18405631579549" />
+        xyz="1.55431223447522E-15 -1.55431223447522E-15 0.1"
+        rpy="0 0 0" />
+      <mass
+        value="42.8421975932662" />
+      <inertia
+        ixx="0.843504879614984"
+        ixy="-9.59503304028305E-33"
+        ixz="6.01287397790472E-17"
+        iyy="0.843504879614984"
+        iyz="-2.42963471245841E-16"
+        izz="1.34196583325215" />
     </inertial>
     <visual>
@@ -305,6 +305,6 @@
     type="continuous">
     <origin
-      xyz="-0.523273265196343 -0.275 0.250000000000001"
-      rpy="1.5707963267949 0 0" />
+      xyz="-0.52327 -0.275 0.25"
+      rpy="1.5708 0 0" />
     <parent
       link="base_link" />
@@ -320,15 +320,15 @@
     <inertial>
       <origin
-        xyz="3.33066907387547E-16 -1.11022302462516E-16 0.0999999999999998"
-        rpy="0 0 0" />
-      <mass
-        value="39.8759403950152" />
-      <inertia
-        ixx="0.738004078739411"
-        ixy="-6.00424777087413E-33"
-        ixz="5.78644975246967E-19"
-        iyy="0.73800407873941"
-        iyz="7.25303828077831E-18"
-        izz="1.18405631579549" />
+        xyz="3.33066907387547E-16 -2.22044604925031E-16 0.0999999999999999"
+        rpy="0 0 0" />
+      <mass
+        value="42.8421975932662" />
+      <inertia
+        ixx="0.843504879614984"
+        ixy="-5.97993043604167E-33"
+        ixz="-3.69567293190445E-18"
+        iyy="0.843504879614984"
+        iyz="1.50156913172873E-17"
+        izz="1.34196583325215" />
     </inertial>
     <visual>
@@ -360,6 +360,6 @@
     type="continuous">
     <origin
-      xyz="-0.523273265196342 0.275 0.249999999999999"
-      rpy="-1.5707963267949 0 0" />
+      xyz="-0.52327 0.275 0.25"
+      rpy="-1.5708 0 0" />
     <parent
       link="base_link" />
@@ -415,5 +415,5 @@
     type="fixed">
     <origin
-      xyz="0.0767267348036579 0 0.63"
+      xyz="0.076727 0 0.63"
       rpy="0 0 0" />
     <parent
@@ -424,3 +424,162 @@
       xyz="0 0 0" />
   </joint>
+  <link
+    name="gps_link">
+    <inertial>
+      <origin
+        xyz="0 0 -0.00999999999999995"
+        rpy="0 0 0" />
+      <mass
+        value="0.1" />
+      <inertia
+        ixx="8.66666666666667E-05"
+        ixy="1.76566841298316E-20"
+        ixz="1.00796920723262E-21"
+        iyy="2.41666666666667E-05"
+        iyz="-4.3548787261501E-22"
+        izz="0.000104166666666667" />
+    </inertial>
+    <visual>
+      <origin
+        xyz="0 0 0"
+        rpy="0 0 0" />
+      <geometry>
+        <mesh
+          filename="package://puma_model/meshes/gps_link.STL" />
+      </geometry>
+      <material
+        name="">
+        <color
+          rgba="0.623529411764706 1 0.76078431372549 1" />
+      </material>
+    </visual>
+    <collision>
+      <origin
+        xyz="0 0 0"
+        rpy="0 0 0" />
+      <geometry>
+        <mesh
+          filename="package://puma_model/meshes/gps_link.STL" />
+      </geometry>
+    </collision>
+  </link>
+  <joint
+    name="gps_joint"
+    type="fixed">
+    <origin
+      xyz="0.22173 0 0.76"
+      rpy="0 0 0" />
+    <parent
+      link="base_link" />
+    <child
+      link="gps_link" />
+    <axis
+      xyz="0 0 0" />
+  </joint>
+  <link
+    name="imu1_link">
+    <inertial>
+      <origin
+        xyz="0.01 0 0"
+        rpy="0 0 0" />
+      <mass
+        value="0.1" />
+      <inertia
+        ixx="0.000104166666666667"
+        ixy="1.57322252736699E-21"
+        ixz="2.01593841446523E-21"
+        iyy="8.6666666666667E-05"
+        iyz="-1.03902708196528E-20"
+        izz="2.41666666666667E-05" />
+    </inertial>
+    <visual>
+      <origin
+        xyz="0 0 0"
+        rpy="0 0 0" />
+      <geometry>
+        <mesh
+          filename="package://puma_model/meshes/imu1_link.STL" />
+      </geometry>
+      <material
+        name="">
+        <color
+          rgba="0.792156862745098 0.819607843137255 0.933333333333333 1" />
+      </material>
+    </visual>
+    <collision>
+      <origin
+        xyz="0 0 0"
+        rpy="0 0 0" />
+      <geometry>
+        <mesh
+          filename="package://puma_model/meshes/imu1_link.STL" />
+      </geometry>
+    </collision>
+  </link>
+  <joint
+    name="imu1_joint"
+    type="fixed">
+    <origin
+      xyz="-0.69327 0 0.57"
+      rpy="0 0 0" />
+    <parent
+      link="base_link" />
+    <child
+      link="imu1_link" />
+    <axis
+      xyz="0 0 0" />
+  </joint>
+  <link
+    name="imu2_link">
+    <inertial>
+      <origin
+        xyz="-0.01 0 0"
+        rpy="0 0 0" />
+      <mass
+        value="0.1" />
+      <inertia
+        ixx="0.000104166666666667"
+        ixy="-5.26402742286973E-22"
+        ixz="2.3628831096606E-21"
+        iyy="8.66666666666669E-05"
+        iyz="6.6181507612138E-22"
+        izz="2.41666666666667E-05" />
+    </inertial>
+    <visual>
+      <origin
+        xyz="0 0 0"
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