Commit message: feat: :sparkles: Change model puma, add camera frame and one imu

File: puma_simulation/puma_model/urdf/puma_model.gazebo.xacro (robot description, xacro)
@@ -23,18 +23,9 @@
     </plugin>
     <!-- Plugin IMU 1 -->
-    <plugin name="imu1_controller" filename="libhector_gazebo_ros_imu.so">
-      <updateRate>30</updateRate>
-      <bodyName>imu1_link</bodyName>
-      <topicName>/imu1</topicName>
-      <frameId>imu1_link</frameId>
-      <gaussianNoise>0 0 0</gaussianNoise>
-      <rpyOffsets>0 0 0</rpyOffsets>
-    </plugin>
-    <!-- Plugin IMU 2  -->
-    <plugin name="imu2_controller" filename="libhector_gazebo_ros_imu.so">
-      <updateRate>30</updateRate>
-      <bodyName>imu2_link</bodyName>
-      <topicName>/imu2</topicName>
-      <frameId>imu2_link</frameId>
+    <plugin name="imu_controller" filename="libhector_gazebo_ros_imu.so">
+      <updateRate>60</updateRate>
+      <bodyName>imu_link</bodyName>
+      <topicName>puma/sensors/imu/raw</topicName>
+      <frameId>imu_link</frameId>
       <gaussianNoise>0 0 0</gaussianNoise>
       <rpyOffsets>0 0 0</rpyOffsets>

File: puma_simulation/puma_model/urdf/puma_model.urdf.xacro (robot description, xacro)
@@ -9,4 +9,529 @@
     <inertial>
       <origin
+        xyz="0.0168277422445081 2.52439420492245E-07 0.369470453921975"
+        rpy="0 0 0" />
+      <mass
+        value="154.381267641272" />
+      <inertia
+        ixx="3.8643546710344"
+        ixy="-9.50231640652348E-07"
+        ixz="1.15363830622366"
+        iyy="22.232099682778"
+        iyz="9.01311880648608E-06"
+        izz="22.6507305397505" />
+    </inertial>
+    <visual>
+      <origin
+        xyz="0 0 0"
+        rpy="0 0 0" />
+      <geometry>
+        <mesh
+          filename="package://puma_model/meshes/base_link.STL" />
+      </geometry>
+      <material
+        name="">
+        <color
+          rgba="0.988235294117647 0.737254901960784 0.517647058823529 1" />
+      </material>
+    </visual>
+    <collision>
+      <origin
+        xyz="0 0 0"
+        rpy="0 0 0" />
+      <geometry>
+        <mesh
+          filename="package://puma_model/meshes/base_link.STL" />
+      </geometry>
+    </collision>
+  </link>
+  <link
+    name="dir_right_link">
+    <inertial>
+      <origin
+        xyz="-2.22044604925031E-16 -0.0294777193153578 1.11022302462516E-16"
+        rpy="0 0 0" />
+      <mass
+        value="0.214607285846125" />
+      <inertia
+        ixx="0.000161787233745492"
+        ixy="-1.25101536732731E-20"
+        ixz="-1.72135905926183E-21"
+        iyy="0.000212842937751498"
+        iyz="1.18540784159886E-20"
+        izz="0.000169651482672632" />
+    </inertial>
+    <visual>
+      <origin
+        xyz="0 0 0"
+        rpy="0 0 0" />
+      <geometry>
+        <mesh
+          filename="package://puma_model/meshes/dir_right_link.STL" />
+      </geometry>
+      <material
+        name="">
+        <color
+          rgba="0.823529411764706 0.823529411764706 0.823529411764706 1" />
+      </material>
+    </visual>
+    <collision>
+      <origin
+        xyz="0 0 0"
+        rpy="0 0 0" />
+      <geometry>
+        <mesh
+          filename="package://puma_model/meshes/dir_right_link.STL" />
+      </geometry>
+    </collision>
+  </link>
+  <joint
+    name="dir_right_joint"
+    type="continuous">
+    <origin
+      xyz="0.576729916214884 -0.337 0.265"
+      rpy="0 0 0" />
+    <parent
+      link="base_link" />
+    <child
+      link="dir_right_link" />
+    <axis
+      xyz="0 0 1" />
+  </joint>
+  <link
+    name="wheel_right_front_link">
+    <inertial>
+      <origin
+        xyz="0 1.11022302462516E-16 0.07"
+        rpy="0 0 0" />
+      <mass
+        value="33.8332405777372" />
+      <inertia
+        ixx="0.663166940004142"
+        ixy="1.74598601904134E-32"
+        ixz="4.51486827425246E-17"
+        iyy="0.663166940004142"
+        iyz="1.07735398960113E-17"
+        izz="1.19194782788173" />
+    </inertial>
+    <visual>
+      <origin
+        xyz="0 0 0"
+        rpy="0 0 0" />
+      <geometry>
+        <mesh
+          filename="package://puma_model/meshes/wheel_right_front_link.STL" />
+      </geometry>
+      <material
+        name="">
+        <color
+          rgba="1 0.752941176470588 0.752941176470588 1" />
+      </material>
+    </visual>
+    <collision>
+      <origin
+        xyz="0 0 0"
+        rpy="0 0 0" />
+      <geometry>
+        <mesh
+          filename="package://puma_model/meshes/wheel_right_front_link.STL" />
+      </geometry>
+    </collision>
+  </link>
+  <joint
+    name="wheel_right_front_joint"
+    type="continuous">
+    <origin
+      xyz="0 -0.048 0"
+      rpy="1.5708 0 0" />
+    <parent
+      link="dir_right_link" />
+    <child
+      link="wheel_right_front_link" />
+    <axis
+      xyz="0 0 -1" />
+    <dynamics
+      friction="1" />
+  </joint>
+  <link
+    name="dir_left_link">
+    <inertial>
+      <origin
+        xyz="0 0.0294777193153578 1.11022302462516E-16"
+        rpy="0 0 0" />
+      <mass
+        value="0.214607285846125" />
+      <inertia
+        ixx="0.000161787233745492"
+        ixy="1.85933047820183E-21"
+        ixz="-2.5363205724219E-21"
+        iyy="0.000212842937751498"
+        iyz="3.87303577600058E-20"
+        izz="0.000169651482672632" />
+    </inertial>
+    <visual>
+      <origin
+        xyz="0 0 0"
+        rpy="0 0 0" />
+      <geometry>
+        <mesh
+          filename="package://puma_model/meshes/dir_left_link.STL" />
+      </geometry>
+      <material
+        name="">
+        <color
+          rgba="0.823529411764706 0.823529411764706 0.823529411764706 1" />
+      </material>
+    </visual>
+    <collision>
+      <origin
+        xyz="0 0 0"
+        rpy="0 0 0" />
+      <geometry>
+        <mesh
+          filename="package://puma_model/meshes/dir_left_link.STL" />
+      </geometry>
+    </collision>
+  </link>
+  <joint
+    name="dir_left_joint"
+    type="continuous">
+    <origin
+      xyz="0.57673 0.337 0.265"
+      rpy="0 0 0" />
+    <parent
+      link="base_link" />
+    <child
+      link="dir_left_link" />
+    <axis
+      xyz="0 0 1" />
+  </joint>
+  <link
+    name="wheel_left_front_link">
+    <inertial>
+      <origin
+        xyz="0 1.11022302462516E-16 0.0699999999999999"
+        rpy="0 0 0" />
+      <mass
+        value="33.8332405777372" />
+      <inertia
+        ixx="0.663166940004142"
+        ixy="3.62902943280336E-32"
+        ixz="-3.47625364951278E-17"
+        iyy="0.663166940004142"
+        iyz="1.01566182105982E-18"
+        izz="1.19194782788173" />
+    </inertial>
+    <visual>
+      <origin
+        xyz="0 0 0"
+        rpy="0 0 0" />
+      <geometry>
+        <mesh
+          filename="package://puma_model/meshes/wheel_left_front_link.STL" />
+      </geometry>
+      <material
+        name="">
+        <color
+          rgba="1 0.752941176470588 0.752941176470588 1" />
+      </material>
+    </visual>
+    <collision>
+      <origin
+        xyz="0 0 0"
+        rpy="0 0 0" />
+      <geometry>
+        <mesh
+          filename="package://puma_model/meshes/wheel_left_front_link.STL" />
+      </geometry>
+    </collision>
+  </link>
+  <joint
+    name="wheel_left_front_joint"
+    type="continuous">
+    <origin
+      xyz="0 0.048 0"
+      rpy="1.5708 0 -3.1416" />
+    <parent
+      link="dir_left_link" />
+    <child
+      link="wheel_left_front_link" />
+    <axis
+      xyz="0 0 -1" />
+    <dynamics
+      friction="1" />
+  </joint>
+  <link
+    name="wheel_right_back_link">
+    <inertial>
+      <origin
+        xyz="0 -1.11022302462516E-16 0.1"
+        rpy="0 0 0" />
+      <mass
+        value="42.8421975932662" />
+      <inertia
+        ixx="0.843504879614984"
+        ixy="-2.17897005442215E-32"
+        ixz="6.01287397790472E-17"
+        iyy="0.843504879614984"
+        iyz="-2.51058847467066E-16"
+        izz="1.34196583325215" />
+    </inertial>
+    <visual>
+      <origin
+        xyz="0 0 0"
+        rpy="0 0 0" />
+      <geometry>
+        <mesh
+          filename="package://puma_model/meshes/wheel_right_back_link.STL" />
+      </geometry>
+      <material
+        name="">
+        <color
+          rgba="0.666666666666667 0.666666666666667 0.666666666666667 1" />
+      </material>
+    </visual>
+    <collision>
+      <origin
+        xyz="0 0 0"
+        rpy="0 0 0" />
+      <geometry>
+        <mesh
+          filename="package://puma_model/meshes/wheel_right_back_link.STL" />
+      </geometry>
+    </collision>
+  </link>
+  <joint
+    name="wheel_right_back_joint"
+    type="continuous">
+    <origin
+      xyz="-0.57327 -0.275 0.25"
+      rpy="1.5708 0 0" />
+    <parent
+      link="base_link" />
+    <child
+      link="wheel_right_back_link" />
+    <axis
+      xyz="0 0 -1" />
+    <dynamics
+      friction="1" />
+  </joint>
+  <link
+    name="wheel_left_back_link">
+    <inertial>
+      <origin
+        xyz="1.11022302462516E-16 1.11022302462516E-16 0.1"
+        rpy="0 0 0" />
+      <mass
+        value="42.8421975932662" />
+      <inertia
+        ixx="0.843504879614984"
+        ixy="-4.06685460585996E-33"
+        ixz="-3.69567293190446E-18"
+        iyy="0.843504879614984"
+        iyz="1.64612942139347E-17"
+        izz="1.34196583325215" />
+    </inertial>
+    <visual>
+      <origin
+        xyz="0 0 0"
+        rpy="0 0 0" />
+      <geometry>
+        <mesh
+          filename="package://puma_model/meshes/wheel_left_back_link.STL" />
+      </geometry>
+      <material
+        name="">
+        <color
+          rgba="0.666666666666667 0.666666666666667 0.666666666666667 1" />
+      </material>
+    </visual>
+    <collision>
+      <origin
+        xyz="0 0 0"
+        rpy="0 0 0" />
+      <geometry>
+        <mesh
+          filename="package://puma_model/meshes/wheel_left_back_link.STL" />
+      </geometry>
+    </collision>
+  </link>
+  <joint
+    name="wheel_left_back_joint"
+    type="continuous">
+    <origin
+      xyz="-0.57327 0.275 0.25"
+      rpy="-1.5708 0 0" />
+    <parent
+      link="base_link" />
+    <child
+      link="wheel_left_back_link" />
+    <axis
+      xyz="0 0 -1" />
+    <dynamics
+      friction="1" />
+  </joint>
+  <link
+    name="base_component_link">
+    <inertial>
+      <origin
+        xyz="-1.3878E-17 -1.3878E-17 0"
+        rpy="0 0 0" />
+      <mass
+        value="26.928" />
+      <inertia
+        ixx="0.39943"
+        ixy="1.537E-18"
+        ixz="-1.0408E-17"
+        iyy="0.36802"
+        iyz="1.0408E-17"
+        izz="0.55023" />
+    </inertial>
+    <visual>
+      <origin
+        xyz="0 0 0"
+        rpy="0 0 0" />
+      <geometry>
+        <mesh
+          filename="package://puma_model/meshes/base_component_link.STL" />
+      </geometry>
+      <material
+        name="">
+        <color
+          rgba="1 0.75294 1 1" />
+      </material>
+    </visual>
+    <collision>
+      <origin
+        xyz="0 0 0"
+        rpy="0 0 0" />
+      <geometry>
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
File: puma_simulation/puma_model_camera/urdf/puma_model.gazebo.xacro (robot description, xacro)
@@ -23,18 +23,9 @@
     </plugin>
     <!-- Plugin IMU 1 -->
-    <plugin name="imu1_controller" filename="libhector_gazebo_ros_imu.so">
-      <updateRate>30</updateRate>
-      <bodyName>imu1_link</bodyName>
-      <topicName>/imu1</topicName>
-      <frameId>imu1_link</frameId>
-      <gaussianNoise>0 0 0</gaussianNoise>
-      <rpyOffsets>0 0 0</rpyOffsets>
-    </plugin>
-    <!-- Plugin IMU 2  -->
-    <plugin name="imu2_controller" filename="libhector_gazebo_ros_imu.so">
-      <updateRate>30</updateRate>
-      <bodyName>imu2_link</bodyName>
-      <topicName>/imu2</topicName>
-      <frameId>imu2_link</frameId>
+    <plugin name="imu_controller" filename="libhector_gazebo_ros_imu.so">
+      <updateRate>60</updateRate>
+      <bodyName>imu_link</bodyName>
+      <topicName>puma/sensors/imu/raw</topicName>
+      <frameId>imu_link</frameId>
       <gaussianNoise>0 0 0</gaussianNoise>
       <rpyOffsets>0 0 0</rpyOffsets>

File: puma_simulation/puma_model_camera/urdf/puma_model.urdf.xacro (robot description, xacro)
@@ -15,4 +15,529 @@
     <inertial>
       <origin
+        xyz="0.0168277422445081 2.52439420492245E-07 0.369470453921975"
+        rpy="0 0 0" />
+      <mass
+        value="154.381267641272" />
+      <inertia
+        ixx="3.8643546710344"
+        ixy="-9.50231640652348E-07"
+        ixz="1.15363830622366"
+        iyy="22.232099682778"
+        iyz="9.01311880648608E-06"
+        izz="22.6507305397505" />
+    </inertial>
+    <visual>
+      <origin
+        xyz="0 0 0"
+        rpy="0 0 0" />
+      <geometry>
+        <mesh
+          filename="package://puma_model/meshes/base_link.STL" />
+      </geometry>
+      <material
+        name="">
+        <color
+          rgba="0.988235294117647 0.737254901960784 0.517647058823529 1" />
+      </material>
+    </visual>
+    <collision>
+      <origin
+        xyz="0 0 0"
+        rpy="0 0 0" />
+      <geometry>
+        <mesh
+          filename="package://puma_model/meshes/base_link.STL" />
+      </geometry>
+    </collision>
+  </link>
+  <link
+    name="dir_right_link">
+    <inertial>
+      <origin
+        xyz="-2.22044604925031E-16 -0.0294777193153578 1.11022302462516E-16"
+        rpy="0 0 0" />
+      <mass
+        value="0.214607285846125" />
+      <inertia
+        ixx="0.000161787233745492"
+        ixy="-1.25101536732731E-20"
+        ixz="-1.72135905926183E-21"
+        iyy="0.000212842937751498"
+        iyz="1.18540784159886E-20"
+        izz="0.000169651482672632" />
+    </inertial>
+    <visual>
+      <origin
+        xyz="0 0 0"
+        rpy="0 0 0" />
+      <geometry>
+        <mesh
+          filename="package://puma_model/meshes/dir_right_link.STL" />
+      </geometry>
+      <material
+        name="">
+        <color
+          rgba="0.823529411764706 0.823529411764706 0.823529411764706 1" />
+      </material>
+    </visual>
+    <collision>
+      <origin
+        xyz="0 0 0"
+        rpy="0 0 0" />
+      <geometry>
+        <mesh
+          filename="package://puma_model/meshes/dir_right_link.STL" />
+      </geometry>
+    </collision>
+  </link>
+  <joint
+    name="dir_right_joint"
+    type="continuous">
+    <origin
+      xyz="0.576729916214884 -0.337 0.265"
+      rpy="0 0 0" />
+    <parent
+      link="base_link" />
+    <child
+      link="dir_right_link" />
+    <axis
+      xyz="0 0 1" />
+  </joint>
+  <link
+    name="wheel_right_front_link">
+    <inertial>
+      <origin
+        xyz="0 1.11022302462516E-16 0.07"
+        rpy="0 0 0" />
+      <mass
+        value="33.8332405777372" />
+      <inertia
+        ixx="0.663166940004142"
+        ixy="1.74598601904134E-32"
+        ixz="4.51486827425246E-17"
+        iyy="0.663166940004142"
+        iyz="1.07735398960113E-17"
+        izz="1.19194782788173" />
+    </inertial>
+    <visual>
+      <origin
+        xyz="0 0 0"
+        rpy="0 0 0" />
+      <geometry>
+        <mesh
+          filename="package://puma_model/meshes/wheel_right_front_link.STL" />
+      </geometry>
+      <material
+        name="">
+        <color
+          rgba="1 0.752941176470588 0.752941176470588 1" />
+      </material>
+    </visual>
+    <collision>
+      <origin
+        xyz="0 0 0"
+        rpy="0 0 0" />
+      <geometry>
+        <mesh
+          filename="package://puma_model/meshes/wheel_right_front_link.STL" />
+      </geometry>
+    </collision>
+  </link>
+  <joint
+    name="wheel_right_front_joint"
+    type="continuous">
+    <origin
+      xyz="0 -0.048 0"
+      rpy="1.5708 0 0" />
+    <parent
+      link="dir_right_link" />
+    <child
+      link="wheel_right_front_link" />
+    <axis
+      xyz="0 0 -1" />
+    <dynamics
+      friction="1" />
+  </joint>
+  <link
+    name="dir_left_link">
+    <inertial>
+      <origin
+        xyz="0 0.0294777193153578 1.11022302462516E-16"
+        rpy="0 0 0" />
+      <mass
+        value="0.214607285846125" />
+      <inertia
+        ixx="0.000161787233745492"
+        ixy="1.85933047820183E-21"
+        ixz="-2.5363205724219E-21"
+        iyy="0.000212842937751498"
+        iyz="3.87303577600058E-20"
+        izz="0.000169651482672632" />
+    </inertial>
+    <visual>
+      <origin
+        xyz="0 0 0"
+        rpy="0 0 0" />
+      <geometry>
+        <mesh
+          filename="package://puma_model/meshes/dir_left_link.STL" />
+      </geometry>
+      <material
+        name="">
+        <color
+          rgba="0.823529411764706 0.823529411764706 0.823529411764706 1" />
+      </material>
+    </visual>
+    <collision>
+      <origin
+        xyz="0 0 0"
+        rpy="0 0 0" />
+      <geometry>
+        <mesh
+          filename="package://puma_model/meshes/dir_left_link.STL" />
+      </geometry>
+    </collision>
+  </link>
+  <joint
+    name="dir_left_joint"
+    type="continuous">
+    <origin
+      xyz="0.57673 0.337 0.265"
+      rpy="0 0 0" />
+    <parent
+      link="base_link" />
+    <child
+      link="dir_left_link" />
+    <axis
+      xyz="0 0 1" />
+  </joint>
+  <link
+    name="wheel_left_front_link">
+    <inertial>
+      <origin
+        xyz="0 1.11022302462516E-16 0.0699999999999999"
+        rpy="0 0 0" />
+      <mass
+        value="33.8332405777372" />
+      <inertia
+        ixx="0.663166940004142"
+        ixy="3.62902943280336E-32"
+        ixz="-3.47625364951278E-17"
+        iyy="0.663166940004142"
+        iyz="1.01566182105982E-18"
+        izz="1.19194782788173" />
+    </inertial>
+    <visual>
+      <origin
+        xyz="0 0 0"
+        rpy="0 0 0" />
+      <geometry>
+        <mesh
+          filename="package://puma_model/meshes/wheel_left_front_link.STL" />
+      </geometry>
+      <material
+        name="">
+        <color
+          rgba="1 0.752941176470588 0.752941176470588 1" />
+      </material>
+    </visual>
+    <collision>
+      <origin
+        xyz="0 0 0"
+        rpy="0 0 0" />
+      <geometry>
+        <mesh
+          filename="package://puma_model/meshes/wheel_left_front_link.STL" />
+      </geometry>
+    </collision>
+  </link>
+  <joint
+    name="wheel_left_front_joint"
+    type="continuous">
+    <origin
+      xyz="0 0.048 0"
+      rpy="1.5708 0 -3.1416" />
+    <parent
+      link="dir_left_link" />
+    <child
+      link="wheel_left_front_link" />
+    <axis
+      xyz="0 0 -1" />
+    <dynamics
+      friction="1" />
+  </joint>
+  <link
+    name="wheel_right_back_link">
+    <inertial>
+      <origin
+        xyz="0 -1.11022302462516E-16 0.1"
+        rpy="0 0 0" />
+      <mass
+        value="42.8421975932662" />
+      <inertia
+        ixx="0.843504879614984"
+        ixy="-2.17897005442215E-32"
+        ixz="6.01287397790472E-17"
+        iyy="0.843504879614984"
+        iyz="-2.51058847467066E-16"
+        izz="1.34196583325215" />
+    </inertial>
+    <visual>
+      <origin
+        xyz="0 0 0"
+        rpy="0 0 0" />
+      <geometry>
+        <mesh
+          filename="package://puma_model/meshes/wheel_right_back_link.STL" />
+      </geometry>
+      <material
+        name="">
+        <color
+          rgba="0.666666666666667 0.666666666666667 0.666666666666667 1" />
+      </material>
+    </visual>
+    <collision>
+      <origin
+        xyz="0 0 0"
+        rpy="0 0 0" />
+      <geometry>
+        <mesh
+          filename="package://puma_model/meshes/wheel_right_back_link.STL" />
+      </geometry>
+    </collision>
+  </link>
+  <joint
+    name="wheel_right_back_joint"
+    type="continuous">
+    <origin
+      xyz="-0.57327 -0.275 0.25"
+      rpy="1.5708 0 0" />
+    <parent
+      link="base_link" />
+    <child
+      link="wheel_right_back_link" />
+    <axis
+      xyz="0 0 -1" />
+    <dynamics
+      friction="1" />
+  </joint>
+  <link
+    name="wheel_left_back_link">
+    <inertial>
+      <origin
+        xyz="1.11022302462516E-16 1.11022302462516E-16 0.1"
+        rpy="0 0 0" />
+      <mass
+        value="42.8421975932662" />
+      <inertia
+        ixx="0.843504879614984"
+        ixy="-4.06685460585996E-33"
+        ixz="-3.69567293190446E-18"
+        iyy="0.843504879614984"
+        iyz="1.64612942139347E-17"
+        izz="1.34196583325215" />
+    </inertial>
+    <visual>
+      <origin
+        xyz="0 0 0"
+        rpy="0 0 0" />
+      <geometry>
+        <mesh
+          filename="package://puma_model/meshes/wheel_left_back_link.STL" />
+      </geometry>
+      <material
+        name="">
+        <color
+          rgba="0.666666666666667 0.666666666666667 0.666666666666667 1" />
+      </material>
+    </visual>
+    <collision>
+      <origin
+        xyz="0 0 0"
+        rpy="0 0 0" />
+      <geometry>
+        <mesh
+          filename="package://puma_model/meshes/wheel_left_back_link.STL" />
+      </geometry>
+    </collision>
+  </link>
+  <joint
+    name="wheel_left_back_joint"
+    type="continuous">
+    <origin
+      xyz="-0.57327 0.275 0.25"
+      rpy="-1.5708 0 0" />
+    <parent
+      link="base_link" />
+    <child
+      link="wheel_left_back_link" />
+    <axis
+      xyz="0 0 -1" />
+    <dynamics
+      friction="1" />
+  </joint>
+  <link
+    name="base_component_link">
+    <inertial>
+      <origin
+        xyz="-1.3878E-17 -1.3878E-17 0"
+        rpy="0 0 0" />
+      <mass
+        value="26.928" />
+      <inertia
+        ixx="0.39943"
+        ixy="1.537E-18"
+        ixz="-1.0408E-17"
+        iyy="0.36802"
+        iyz="1.0408E-17"
+        izz="0.55023" />
+    </inertial>
+    <visual>
+      <origin
+        xyz="0 0 0"
+        rpy="0 0 0" />
+      <geometry>
+        <mesh
+          filename="package://puma_model/meshes/base_component_link.STL" />
+      </geometry>
+      <material
+        name="">
+        <color
+          rgba="1 0.75294 1 1" />
+      </material>
+    </visual>
+    <collision>
+      <origin
+        xyz="0 0 0"
+        rpy="0 0 0" />
+      <geometry>
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