Commit message: Fix minor bug

File: puma_simulation/puma_model_camera/urdf/d455.urdf.xacro (robot description, xacro)
@@ -56,5 +56,5 @@
         <geometry>
           <!-- <box size="${d455_cam_depth} ${d455_cam_width} ${d455_cam_height}"/> -->
-	        <mesh filename="package://example_simulation_camera/meshes/d455.stl" scale="0.001 0.001 0.001" />
+	        <mesh filename="package://puma_model_camera/meshes/d455.stl" scale="0.001 0.001 0.001" />
         </geometry>
         <material name="aluminum"/>
