Commit message: feat: :construction: Work in puma local planner and add model with change in base link

File: puma_simulation/puma_model_camera/urdf/puma_model.urdf.xacro (robot description, xacro)
@@ -3,5 +3,5 @@
      Commit Version: 1.6.0-4-g7f85cfe  Build Version: 1.6.7995.38578
      For more information, please see http://wiki.ros.org/sw_urdf_exporter -->
-<robot name="puma_model" xmlns:xacro="http://ros.org/wiki/xacro">
+<robot name="puma_model_camera" xmlns:xacro="http://ros.org/wiki/xacro">
   <xacro:include filename="$(find puma_model_camera)/urdf/puma_model.gazebo.xacro"/>
   <xacro:arg name="use_nominal_extrinsics" default="true"/>
@@ -15,5 +15,5 @@
     <inertial>
       <origin
-        xyz="0.0168277422445081 2.52439420492245E-07 0.369470453921975"
+        xyz="0.590095933243336 2.52439420506123E-07 0.369470453921976"
         rpy="0 0 0" />
       <mass
@@ -21,8 +21,8 @@
       <inertia
         ixx="3.8643546710344"
-        ixy="-9.50231640652348E-07"
+        ixy="-9.50231640653173E-07"
         ixz="1.15363830622366"
         iyy="22.232099682778"
-        iyz="9.01311880648608E-06"
+        iyz="9.01311880647381E-06"
         izz="22.6507305397505" />
     </inertial>
@@ -33,5 +33,5 @@
       <geometry>
         <mesh
-          filename="package://puma_model/meshes/base_link.STL" />
+          filename="package://puma_model_camera/meshes/base_link.STL" />
       </geometry>
       <material
@@ -47,5 +47,5 @@
       <geometry>
         <mesh
-          filename="package://puma_model/meshes/base_link.STL" />
+          filename="package://puma_model_camera/meshes/base_link.STL" />
       </geometry>
     </collision>
@@ -61,8 +61,8 @@
       <inertia
         ixx="0.000161787233745492"
-        ixy="-1.25101536732731E-20"
-        ixz="-1.72135905926183E-21"
+        ixy="-1.25429054904435E-20"
+        ixz="-1.78299811249943E-21"
         iyy="0.000212842937751498"
-        iyz="1.18540784159886E-20"
+        iyz="1.23372093603248E-20"
         izz="0.000169651482672632" />
     </inertial>
@@ -73,5 +73,5 @@
       <geometry>
         <mesh
-          filename="package://puma_model/meshes/dir_right_link.STL" />
+          filename="package://puma_model_camera/meshes/dir_right_link.STL" />
       </geometry>
       <material
@@ -87,5 +87,5 @@
       <geometry>
         <mesh
-          filename="package://puma_model/meshes/dir_right_link.STL" />
+          filename="package://puma_model_camera/meshes/dir_right_link.STL" />
       </geometry>
     </collision>
@@ -95,5 +95,5 @@
     type="continuous">
     <origin
-      xyz="0.576729916214884 -0.337 0.265"
+      xyz="1.15 -0.337 0.265"
       rpy="0 0 0" />
     <parent
@@ -126,5 +126,5 @@
       <geometry>
         <mesh
-          filename="package://puma_model/meshes/wheel_right_front_link.STL" />
+          filename="package://puma_model_camera/meshes/wheel_right_front_link.STL" />
       </geometry>
       <material
@@ -140,5 +140,5 @@
       <geometry>
         <mesh
-          filename="package://puma_model/meshes/wheel_right_front_link.STL" />
+          filename="package://puma_model_camera/meshes/wheel_right_front_link.STL" />
       </geometry>
     </collision>
@@ -169,8 +169,8 @@
       <inertia
         ixx="0.000161787233745492"
-        ixy="1.85933047820183E-21"
-        ixz="-2.5363205724219E-21"
+        ixy="1.44494928036241E-21"
+        ixz="-2.86590106719918E-21"
         iyy="0.000212842937751498"
-        iyz="3.87303577600058E-20"
+        iyz="2.66957117537751E-20"
         izz="0.000169651482672632" />
     </inertial>
@@ -181,5 +181,5 @@
       <geometry>
         <mesh
-          filename="package://puma_model/meshes/dir_left_link.STL" />
+          filename="package://puma_model_camera/meshes/dir_left_link.STL" />
       </geometry>
       <material
@@ -195,5 +195,5 @@
       <geometry>
         <mesh
-          filename="package://puma_model/meshes/dir_left_link.STL" />
+          filename="package://puma_model_camera/meshes/dir_left_link.STL" />
       </geometry>
     </collision>
@@ -203,5 +203,5 @@
     type="continuous">
     <origin
-      xyz="0.57673 0.337 0.265"
+      xyz="1.15 0.337 0.265"
       rpy="0 0 0" />
     <parent
@@ -216,5 +216,5 @@
     <inertial>
       <origin
-        xyz="0 1.11022302462516E-16 0.0699999999999999"
+        xyz="0 0 0.0699999999999999"
         rpy="0 0 0" />
       <mass
@@ -234,5 +234,5 @@
       <geometry>
         <mesh
-          filename="package://puma_model/meshes/wheel_left_front_link.STL" />
+          filename="package://puma_model_camera/meshes/wheel_left_front_link.STL" />
       </geometry>
       <material
@@ -248,5 +248,5 @@
       <geometry>
         <mesh
-          filename="package://puma_model/meshes/wheel_left_front_link.STL" />
+          filename="package://puma_model_camera/meshes/wheel_left_front_link.STL" />
       </geometry>
     </collision>
@@ -289,5 +289,5 @@
       <geometry>
         <mesh
-          filename="package://puma_model/meshes/wheel_right_back_link.STL" />
+          filename="package://puma_model_camera/meshes/wheel_right_back_link.STL" />
       </geometry>
       <material
@@ -303,5 +303,5 @@
       <geometry>
         <mesh
-          filename="package://puma_model/meshes/wheel_right_back_link.STL" />
+          filename="package://puma_model_camera/meshes/wheel_right_back_link.STL" />
       </geometry>
     </collision>
@@ -311,5 +311,5 @@
     type="continuous">
     <origin
-      xyz="-0.57327 -0.275 0.25"
+      xyz="0 -0.275 0.25"
       rpy="1.5708 0 0" />
     <parent
@@ -332,5 +332,5 @@
       <inertia
         ixx="0.843504879614984"
-        ixy="-4.06685460585996E-33"
+        ixy="-4.06685460585995E-33"
         ixz="-3.69567293190446E-18"
         iyy="0.843504879614984"
@@ -344,5 +344,5 @@
       <geometry>
         <mesh
-          filename="package://puma_model/meshes/wheel_left_back_link.STL" />
+          filename="package://puma_model_camera/meshes/wheel_left_back_link.STL" />
       </geometry>
       <material
@@ -358,5 +358,5 @@
       <geometry>
         <mesh
-          filename="package://puma_model/meshes/wheel_left_back_link.STL" />
+          filename="package://puma_model_camera/meshes/wheel_left_back_link.STL" />
       </geometry>
     </collision>
@@ -366,5 +366,5 @@
     type="continuous">
     <origin
-      xyz="-0.57327 0.275 0.25"
+      xyz="0 0.275 0.25"
       rpy="-1.5708 0 0" />
     <parent
@@ -381,37 +381,37 @@
     <inertial>
       <origin
-        xyz="-1.3878E-17 -1.3878E-17 0"
+        xyz="-1.38777878078145E-17 -1.38777878078145E-17 0"
         rpy="0 0 0" />
       <mass
         value="26.928" />
       <inertia
-        ixx="0.39943"
-        ixy="1.537E-18"
-        ixz="-1.0408E-17"
-        iyy="0.36802"
-        iyz="1.0408E-17"
-        izz="0.55023" />
-    </inertial>
-    <visual>
-      <origin
-        xyz="0 0 0"
-        rpy="0 0 0" />
-      <geometry>
-        <mesh
-          filename="package://puma_model/meshes/base_component_link.STL" />
-      </geometry>
-      <material
-        name="">
-        <color
-          rgba="1 0.75294 1 1" />
-      </material>
-    </visual>
-    <collision>
-      <origin
-        xyz="0 0 0"
-        rpy="0 0 0" />
-      <geometry>
-        <mesh
-          filename="package://puma_model/meshes/base_component_link.STL" />
+        ixx="0.399432"
+        ixy="1.53695574785691E-18"
+        ixz="-1.04083408558608E-17"
+        iyy="0.368016"
+        iyz="1.04083408558608E-17"
+        izz="0.5502288" />
+    </inertial>
+    <visual>
+      <origin
+        xyz="0 0 0"
+        rpy="0 0 0" />
+      <geometry>
+        <mesh
+          filename="package://puma_model_camera/meshes/base_component_link.STL" />
+      </geometry>
+      <material
+        name="">
+        <color
+          rgba="1 0.752941176470588 1 1" />
+      </material>
+    </visual>
+    <collision>
+      <origin
+        xyz="0 0 0"
+        rpy="0 0 0" />
+      <geometry>
+        <mesh
+          filename="package://puma_model_camera/meshes/base_component_link.STL" />
       </geometry>
     </collision>
@@ -421,5 +421,5 @@
     type="fixed">
     <origin
-      xyz="0.12673 0 0.63"
+      xyz="0.7 0 0.63"
       rpy="0 0 0" />
     <parent
@@ -434,37 +434,37 @@
     <inertial>
       <origin
-        xyz="0 -1.3878E-17 -0.01"
+        xyz="0 -1.38777878078145E-17 -0.01"
         rpy="0 0 0" />
       <mass
         value="0.1" />
       <inertia
-        ixx="8.6667E-05"
-        ixy="7.1603E-22"
-        ixz="1.084E-37"
-        iyy="2.4167E-05"
-        iyz="-4.3549E-22"
-        izz="0.00010417" />
-    </inertial>
-    <visual>
-      <origin
-        xyz="0 0 0"
-        rpy="0 0 0" />
-      <geometry>
-        <mesh
-          filename="package://puma_model/meshes/gps_link.STL" />
-      </geometry>
-      <material
-        name="">
-        <color
-          rgba="0.62353 1 0.76078 1" />
-      </material>
-    </visual>
-    <collision>
-      <origin
-        xyz="0 0 0"
-        rpy="0 0 0" />
-      <geometry>
-        <mesh
-          filename="package://puma_model/meshes/gps_link.STL" />
+        ixx="8.66666666666668E-05"
+        ixy="-6.77626357803215E-24"
+        ixz="9.37383128294732E-23"
+        iyy="2.41666666666667E-05"
+        iyz="-2.17743936307505E-22"
+        izz="0.000104166666666667" />
+    </inertial>
+    <visual>
+      <origin
+        xyz="0 0 0"
+        rpy="0 0 0" />
+      <geometry>
+        <mesh
+          filename="package://puma_model_camera/meshes/gps_link.STL" />
+      </geometry>
+      <material
+        name="">
+        <color
+          rgba="0.623529411764706 1 0.76078431372549 1" />
+      </material>
+    </visual>
+    <collision>
+      <origin
+        xyz="0 0 0"
+        rpy="0 0 0" />
+      <geometry>
+        <mesh
+          filename="package://puma_model_camera/meshes/gps_link.STL" />
       </geometry>
     </collision>
@@ -474,5 +474,5 @@
     type="fixed">
     <origin
-      xyz="0.27173 0 0.76"
+      xyz="0.845 0 0.76"
       rpy="0 0 0" />
     <parent
@@ -487,37 +487,37 @@
     <inertial>
       <origin
-        xyz="5.0806E-07 -0.00019557 -0.012163"
-        rpy="0 0 0" />
-      <mass
-        value="0.010655" />
-      <inertia
-        ixx="1.1671E-06"
-        ixy="2.0326E-11"
-        ixz="2.1164E-12"
-        iyy="2.2054E-06"
-        iyz="-8.1469E-10"
-        izz="2.7832E-06" />
-    </inertial>
-    <visual>
-      <origin
-        xyz="0 0 0"
-        rpy="0 0 0" />
-      <geometry>
-        <mesh
-          filename="package://puma_model/meshes/imu_link.STL" />
-      </geometry>
-      <material
-        name="">
-        <color
-          rgba="0.79216 0.81961 0.93333 1" />
-      </material>
-    </visual>
-    <collision>
-      <origin
-        xyz="0 0 0"
-        rpy="0 0 0" />
-      <geometry>
-        <mesh
-          filename="package://puma_model/meshes/imu_link.STL" />
+        xyz="5.08055300330046E-07 -0.000195569944066137 -0.0121628383871962"
+        rpy="0 0 0" />
+      <mass
+        value="0.0106550387325199" />
+      <inertia
+        ixx="1.16705248203446E-06"
+        ixy="2.03256158405584E-11"
+        ixz="2.1164211381414E-12"
+        iyy="2.20541869708662E-06"
+        iyz="-8.14691556822219E-10"
+        izz="2.78315231388432E-06" />
+    </inertial>
+    <visual>
+      <origin
+        xyz="0 0 0"
+        rpy="0 0 0" />
+      <geometry>
+        <mesh
+          filename="package://puma_model_camera/meshes/imu_link.STL" />
+      </geometry>
+      <material
+        name="">
+        <color
+          rgba="0.792156862745098 0.819607843137255 0.933333333333333 1" />
+      </material>
+    </visual>
+    <collision>
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